Commit message: "Finished quadruped"

File: body.urdf (robot description, URDF)
Before this commit: robot robot, 3 links, 2 joints
Links:
- added link BLowerLeg, mass 1; collision box size=0.2 0.2 1; visual box size=0.2 0.2 1
- added link FLowerLeg, mass 1; collision box size=0.2 0.2 1; visual box size=0.2 0.2 1
- added link LLowerLeg, mass 1; collision box size=0.2 0.2 1; visual box size=0.2 0.2 1
- added link LeftLeg, mass 1; collision box size=1 0.2 0.2; visual box size=1 0.2 0.2
- added link RLowerLeg, mass 1; collision box size=0.2 0.2 1; visual box size=0.2 0.2 1
- added link RightLeg, mass 1; collision box size=1 0.2 0.2; visual box size=1 0.2 0.2
- link BackLeg: geometry collision box size=0.2 1 0.2; visual box size=0.2 1 0.2
- link FrontLeg: geometry collision box size=0.2 1 0.2; visual box size=0.2 1 0.2
Joints:
- added joint BackLeg_BLowerLeg: type revolute, parent BackLeg, child BLowerLeg, origin xyz=0 -1 0 rpy=0 0 0, axis 1 0 0, limit lower=-3.14159 upper=3.14159 effort=0.0 velocity=0.0
- added joint FrontLeg_FLowerLeg: type revolute, parent FrontLeg, child FLowerLeg, origin xyz=0 1 0 rpy=0 0 0, axis 1 0 0, limit lower=-3.14159 upper=3.14159 effort=0.0 velocity=0.0
- added joint LeftLeg_LLowerLeg: type revolute, parent LeftLeg, child LLowerLeg, origin xyz=-1 0 0 rpy=0 0 0, axis 0 1 0, limit lower=-3.14159 upper=3.14159 effort=0.0 velocity=0.0
- added joint RightLeg_RLowerLeg: type revolute, parent RightLeg, child RLowerLeg, origin xyz=1 0 0 rpy=0 0 0, axis 0 1 0, limit lower=-3.14159 upper=3.14159 effort=0.0 velocity=0.0
- added joint Torso_LeftLeg: type revolute, parent Torso, child LeftLeg, origin xyz=-0.5 0 1 rpy=0 0 0, axis 0 1 0, limit lower=-3.14159 upper=3.14159 effort=0.0 velocity=0.0
- added joint Torso_RightLeg: type revolute, parent Torso, child RightLeg, origin xyz=0.5 0 1 rpy=0 0 0, axis 0 1 0, limit lower=-3.14159 upper=3.14159 effort=0.0 velocity=0.0
- joint Torso_BackLeg: axis 0 1 0 -> 1 0 0; origin xyz=1 0 1 rpy=0 0 0 -> xyz=0 -0.5 1 rpy=0 0 0
- joint Torso_FrontLeg: axis 0 1 0 -> 1 0 0; origin xyz=2 0 1 rpy=0 0 0 -> xyz=0 0.5 1 rpy=0 0 0

Commit message: "Finished Asn 5"

File: body.urdf (robot description, URDF)
Before this commit: robot robot, 9 links, 8 joints
Links:
- removed link BLowerLeg
- removed link BackLeg
- removed link FLowerLeg
- removed link FrontLeg
- removed link LLowerLeg
- removed link LeftLeg
- removed link RLowerLeg
- removed link RightLeg
- added link LArm, mass 1; collision box size=0.3 0.3 0.8; visual box size=0.3 0.3 0.8
- added link LShin, mass 1; collision box size=0.3 0.3 0.7; visual box size=0.3 0.3 0.7
- added link LThigh, mass 1; collision box size=0.3 0.3 0.6; visual box size=0.3 0.3 0.6
- added link RArm, mass 1; collision box size=0.3 0.3 0.8; visual box size=0.3 0.3 0.8
- added link RShin, mass 1; collision box size=0.3 0.3 0.7; visual box size=0.3 0.3 0.7
- added link RThigh, mass 1; collision box size=0.3 0.3 0.6; visual box size=0.3 0.3 0.6
- link Torso: geometry collision box size=0.5 0.8 1; visual box size=0.5 0.8 1
Joints:
- removed joint BackLeg_BLowerLeg
- removed joint FrontLeg_FLowerLeg
- removed joint LeftLeg_LLowerLeg
- removed joint RightLeg_RLowerLeg
- removed joint Torso_BackLeg
- removed joint Torso_FrontLeg
- removed joint Torso_LeftLeg
- removed joint Torso_RightLeg
- added joint LThigh_LShin: type revolute, parent LThigh, child LShin, origin xyz=0 0 -0.6 rpy=0 0 0, axis 0 1 0, limit lower=-3.14159 upper=3.14159 effort=0.0 velocity=0.0
- added joint RThigh_RShin: type revolute, parent RThigh, child RShin, origin xyz=0 0 -0.6 rpy=0 0 0, axis 0 1 0, limit lower=-3.14159 upper=3.14159 effort=0.0 velocity=0.0
- added joint Torso_LArm: type revolute, parent Torso, child LArm, origin xyz=0 -0.4 2.15 rpy=0 0 0, axis 0 1 0, limit lower=-3.14159 upper=3.14159 effort=0.0 velocity=0.0
- added joint Torso_LThigh: type revolute, parent Torso, child LThigh, origin xyz=0 -0.35 1.3 rpy=0 0 0, axis 0 1 0, limit lower=-3.14159 upper=3.14159 effort=0.0 velocity=0.0
- added joint Torso_RArm: type revolute, parent Torso, child RArm, origin xyz=0 0.4 2.15 rpy=0 0 0, axis 0 1 0, limit lower=-3.14159 upper=3.14159 effort=0.0 velocity=0.0
- added joint Torso_RThigh: type revolute, parent Torso, child RThigh, origin xyz=0 0.35 1.3 rpy=0 0 0, axis 0 1 0, limit lower=-3.14159 upper=3.14159 effort=0.0 velocity=0.0

Commit message: "Finished Asn 5"

File: body.urdf (robot description, URDF)
Before this commit: robot robot, 7 links, 6 joints
Links:
- removed link LShin
- removed link RShin
- added link LShank, mass 1; collision box size=0.3 0.3 0.7; visual box size=0.3 0.3 0.7
- added link RShank, mass 1; collision box size=0.3 0.3 0.7; visual box size=0.3 0.3 0.7
Joints:
- removed joint LThigh_LShin
- removed joint RThigh_RShin
- added joint LThigh_LShank: type revolute, parent LThigh, child LShank, origin xyz=0 0 -0.6 rpy=0 0 0, axis 0 1 0, limit lower=-3.14159 upper=3.14159 effort=0.0 velocity=0.0
- added joint RThigh_RShank: type revolute, parent RThigh, child RShank, origin xyz=0 0 -0.6 rpy=0 0 0, axis 0 1 0, limit lower=-3.14159 upper=3.14159 effort=0.0 velocity=0.0

Commit message: "Finished Asn 6"

File: body.urdf (robot description, URDF)
Before this commit: robot robot, 7 links, 6 joints
Links:
- removed link LArm
- removed link LShank
- removed link LThigh
- removed link RArm
- removed link RShank
- removed link RThigh
- removed link Torso
- added link 0, mass 1; collision box size=0.46972307436651284 0.2952829802058358 0.7509863909898356; visual box size=0.46972307436651284 0.2952829802058358 0.7509863909898356
- added link 1, mass 1; collision box size=0.7808400391006156 1.340688094344731 0.482368590269124; visual box size=0.7808400391006156 1.340688094344731 0.482368590269124
- added link 2, mass 1; collision box size=0.9815835206501595 0.8491143614732024 0.7382437324187903; visual box size=0.9815835206501595 0.8491143614732024 0.7382437324187903
- added link 3, mass 1; collision box size=0.2610967851468843 0.3987199690351789 0.8922857931085479; visual box size=0.2610967851468843 0.3987199690351789 0.8922857931085479
- added link 4, mass 1; collision box size=0.6168376170760992 0.8541242653985055 0.8003239336754413; visual box size=0.6168376170760992 0.8541242653985055 0.8003239336754413
- added link 5, mass 1; collision box size=0.3567493415289151 0.7038455571222628 0.47315356386772583; visual box size=0.3567493415289151 0.7038455571222628 0.47315356386772583
- added link 6, mass 1; collision box size=0.6843357216931995 0.26678878957314067 0.5301369538948061; visual box size=0.6843357216931995 0.26678878957314067 0.5301369538948061
- added link 7, mass 1; collision box size=0.31677729205374794 0.6383481501521531 0.7025317200141113; visual box size=0.31677729205374794 0.6383481501521531 0.7025317200141113
Joints:
- removed joint LThigh_LShank
- removed joint RThigh_RShank
- removed joint Torso_LArm
- removed joint Torso_LThigh
- removed joint Torso_RArm
- removed joint Torso_RThigh
- added joint 0_1: type revolute, parent 0, child 1, origin xyz=0 0.1476414901029179 0.5754931954949178 rpy=0 0 0, axis 0 0 1, limit lower=-3.14159 upper=3.14159 effort=0.0 velocity=0.0
- added joint 1_2: type revolute, parent 1, child 2, origin xyz=0 1.340688094344731 0 rpy=0 0 0, axis 0 0 1, limit lower=-3.14159 upper=3.14159 effort=0.0 velocity=0.0
- added joint 2_3: type revolute, parent 2, child 3, origin xyz=0 0.8491143614732024 0 rpy=0 0 0, axis 0 0 1, limit lower=-3.14159 upper=3.14159 effort=0.0 velocity=0.0
- added joint 3_4: type revolute, parent 3, child 4, origin xyz=0 0.3987199690351789 0 rpy=0 0 0, axis 0 0 1, limit lower=-3.14159 upper=3.14159 effort=0.0 velocity=0.0
- added joint 4_5: type revolute, parent 4, child 5, origin xyz=0 0.8541242653985055 0 rpy=0 0 0, axis 0 0 1, limit lower=-3.14159 upper=3.14159 effort=0.0 velocity=0.0
- added joint 5_6: type revolute, parent 5, child 6, origin xyz=0 0.7038455571222628 0 rpy=0 0 0, axis 0 0 1, limit lower=-3.14159 upper=3.14159 effort=0.0 velocity=0.0
- added joint 6_7: type revolute, parent 6, child 7, origin xyz=0 0.26678878957314067 0 rpy=0 0 0, axis 0 0 1, limit lower=-3.14159 upper=3.14159 effort=0.0 velocity=0.0

Commit message: "Finished Asn 6"

File: body.urdf (robot description, URDF)
Before this commit: robot robot, 8 links, 7 joints
Links:
- removed link 5
- removed link 6
- removed link 7
- link 0: geometry collision box size=0.7171555616767803 0.35911951490362526 0.264180151915893; visual box size=0.7171555616767803 0.35911951490362526 0.264180151915893
- link 1: geometry collision box size=0.2574810300310185 1.0157404120389069 0.5954594774265642; visual box size=0.2574810300310185 1.0157404120389069 0.5954594774265642
- link 2: geometry collision box size=0.29167153495723364 0.7299798532252845 0.2735734456196871; visual box size=0.29167153495723364 0.7299798532252845 0.2735734456196871
- link 3: geometry collision box size=0.31699013497129586 0.8473779509513113 0.6980364824096592; visual box size=0.31699013497129586 0.8473779509513113 0.6980364824096592
- link 4: geometry collision box size=0.2767134157820279 0.286300549476845 0.6479783589287489; visual box size=0.2767134157820279 0.286300549476845 0.6479783589287489
Joints:
- removed joint 4_5
- removed joint 5_6
- removed joint 6_7
- joint 0_1: origin xyz=0 0.1476414901029179 0.5754931954949178 rpy=0 0 0 -> xyz=0 0.17955975745181263 0.3320900759579465 rpy=0 0 0
- joint 1_2: origin xyz=0 1.340688094344731 0 rpy=0 0 0 -> xyz=0 1.0157404120389069 0 rpy=0 0 0
- joint 2_3: origin xyz=0 0.8491143614732024 0 rpy=0 0 0 -> xyz=0 0.7299798532252845 0 rpy=0 0 0
- joint 3_4: origin xyz=0 0.3987199690351789 0 rpy=0 0 0 -> xyz=0 0.8473779509513113 0 rpy=0 0 0

Commit message: "Finished Asn 7"

File: body.urdf (robot description, URDF)
Before this commit: robot robot, 5 links, 4 joints
Links:
- added link 10, mass 1; collision box size=0.4300300474687399 0.3960005351491409 0.320397213992056; visual box size=0.4300300474687399 0.3960005351491409 0.320397213992056
- added link 11, mass 1; collision box size=0.2616050874986382 0.4039267225356613 0.4033188927729888; visual box size=0.2616050874986382 0.4039267225356613 0.4033188927729888
- added link 12, mass 1; collision box size=0.2676753044692196 0.17034108154917674 0.19527255188186327; visual box size=0.2676753044692196 0.17034108154917674 0.19527255188186327
- added link 13, mass 1; collision box size=0.4024144216837948 0.24135257212017588 0.41577706259947567; visual box size=0.4024144216837948 0.24135257212017588 0.41577706259947567
- added link 14, mass 1; collision box size=0.4310638551721963 0.38920138744612487 0.2625682432754224; visual box size=0.4310638551721963 0.38920138744612487 0.2625682432754224
- added link 15, mass 1; collision box size=0.14776010378154794 0.19243553305967032 0.15996495766438984; visual box size=0.14776010378154794 0.19243553305967032 0.15996495766438984
- added link 5, mass 1; collision box size=0.4359955126563373 0.23550584780021525 0.43779855136645685; visual box size=0.4359955126563373 0.23550584780021525 0.43779855136645685
- added link 6, mass 1; collision box size=0.1734933875268848 0.27005614426738866 0.2502072442981145; visual box size=0.1734933875268848 0.27005614426738866 0.2502072442981145
- added link 7, mass 1; collision box size=0.3063078888664433 0.3648599756582196 0.2517353929697169; visual box size=0.3063078888664433 0.3648599756582196 0.2517353929697169
- added link 8, mass 1; collision box size=0.2413949467959643 0.42683715933719335 0.4305377879622892; visual box size=0.2413949467959643 0.42683715933719335 0.4305377879622892
- added link 9, mass 1; collision box size=0.21827369318396914 0.21717080818551102 0.18967117007113332; visual box size=0.21827369318396914 0.21717080818551102 0.18967117007113332
- link 0: geometry collision box size=0.5851124687466642 0.31242296501390354 0.5594761066885567; visual box size=0.5851124687466642 0.31242296501390354 0.5594761066885567
- link 1: geometry collision box size=0.3628604417647888 0.3415520305336535 0.25974118535768115; visual box size=0.3628604417647888 0.3415520305336535 0.25974118535768115
- link 2: geometry collision box size=0.2783603214504271 0.3219395401122066 0.2738203385106744; visual box size=0.2783603214504271 0.3219395401122066 0.2738203385106744
- link 3: geometry collision box size=0.2649899806875496 0.18109436189685835 0.26851990878547294; visual box size=0.2649899806875496 0.18109436189685835 0.26851990878547294
- link 4: geometry collision box size=0.24666581848138486 0.24301260928841395 0.2978146028015872; visual box size=0.24666581848138486 0.24301260928841395 0.2978146028015872
Joints:
- removed joint 3_4
- added joint 0_10: type revolute, parent 0, child 10, origin xyz=0 0 2.2797380533442784 rpy=0 0 0, axis 0 0 1, limit lower=-3.14159 upper=3.14159 effort=0.0 velocity=0.0
- added joint 0_13: type revolute, parent 0, child 13, origin xyz=0 0 1.7202619466557216 rpy=0 0 0, axis 1 0 0, limit lower=-3.14159 upper=3.14159 effort=0.0 velocity=0.0
- added joint 0_4: type revolute, parent 0, child 4, origin xyz=0 0.15621148250695177 2 rpy=0 0 0, axis 0 1 0, limit lower=-3.14159 upper=3.14159 effort=0.0 velocity=0.0
- added joint 0_7: type revolute, parent 0, child 7, origin xyz=0 -0.15621148250695177 2 rpy=0 0 0, axis 1 0 0, limit lower=-3.14159 upper=3.14159 effort=0.0 velocity=0.0
- added joint 10_11: type revolute, parent 10, child 11, origin xyz=0 0 0.320397213992056 rpy=0 0 0, axis 1 0 0, limit lower=-3.14159 upper=3.14159 effort=0.0 velocity=0.0
- added joint 11_12: type revolute, parent 11, child 12, origin xyz=0.1308025437493191 0 0.2016594463864944 rpy=0 0 0, axis 1 0 0, limit lower=-3.14159 upper=3.14159 effort=0.0 velocity=0.0
- added joint 13_14: type revolute, parent 13, child 14, origin xyz=0 0 -0.41577706259947567 rpy=0 0 0, axis 0 0 1, limit lower=-3.14159 upper=3.14159 effort=0.0 velocity=0.0
- added joint 14_15: type revolute, parent 14, child 15, origin xyz=0.21553192758609815 0 -0.1312841216377112 rpy=0 0 0, axis 0 0 1, limit lower=-3.14159 upper=3.14159 effort=0.0 velocity=0.0
- added joint 4_5: type revolute, parent 4, child 5, origin xyz=0 0.24301260928841395 0 rpy=0 0 0, axis 0 0 1, limit lower=-3.14159 upper=3.14159 effort=0.0 velocity=0.0
- added joint 5_6: type revolute, parent 5, child 6, origin xyz=0 0.23550584780021525 0 rpy=0 0 0, axis 1 0 0, limit lower=-3.14159 upper=3.14159 effort=0.0 velocity=0.0
- added joint 7_8: type revolute, parent 7, child 8, origin xyz=0 -0.3648599756582196 0 rpy=0 0 0, axis 1 0 0, limit lower=-3.14159 upper=3.14159 effort=0.0 velocity=0.0
- added joint 8_9: type revolute, parent 8, child 9, origin xyz=0 -0.42683715933719335 0 rpy=0 0 0, axis 0 1 0, limit lower=-3.14159 upper=3.14159 effort=0.0 velocity=0.0
- joint 0_1: axis 0 0 1 -> 0 1 0; origin xyz=0 0.17955975745181263 0.3320900759579465 rpy=0 0 0 -> xyz=0.2925562343733321 0 2 rpy=0 0 0
- joint 1_2: axis 0 0 1 -> 0 1 0; origin xyz=0 1.0157404120389069 0 rpy=0 0 0 -> xyz=0.3628604417647888 0 0 rpy=0 0 0
- joint 2_3: axis 0 0 1 -> 0 1 0; origin xyz=0 0.7299798532252845 0 rpy=0 0 0 -> xyz=0.13918016072521355 0 0.1369101692553372 rpy=0 0 0

Commit message: "Finished Asn 7"

File: body.urdf (robot description, URDF)
Before this commit: robot robot, 16 links, 15 joints
Links:
- removed link 10
- removed link 11
- removed link 12
- removed link 13
- removed link 14
- removed link 15
- link 0: geometry collision box size=0.646908251444877 0.6065845087066234 0.5833558861945244; visual box size=0.646908251444877 0.6065845087066234 0.5833558861945244
- link 1: geometry collision box size=0.37282429908884995 0.3537907934278602 0.38473398611796117; visual box size=0.37282429908884995 0.3537907934278602 0.38473398611796117
- link 2: geometry collision box size=0.34618410428685775 0.25624297934783463 0.37431993926747353; visual box size=0.34618410428685775 0.25624297934783463 0.37431993926747353
- link 3: geometry collision box size=0.4027057677449959 0.24653848640400572 0.40075797297576266; visual box size=0.4027057677449959 0.24653848640400572 0.40075797297576266
- link 4: geometry collision box size=0.3997141447006303 0.30909037046842985 0.37616395454667173; visual box size=0.3997141447006303 0.30909037046842985 0.37616395454667173
- link 5: geometry collision box size=0.14642590385519932 0.17425143225345946 0.1850532313059122; visual box size=0.14642590385519932 0.17425143225345946 0.1850532313059122
- link 6: geometry collision box size=0.32644464759038094 0.41319882834782423 0.34599158900683674; visual box size=0.32644464759038094 0.41319882834782423 0.34599158900683674
- link 7: geometry collision box size=0.2443913508406264 0.23689179907693925 0.32704650887761855; visual box size=0.2443913508406264 0.23689179907693925 0.32704650887761855
- link 8: geometry collision box size=0.3576547495187927 0.31346256494802144 0.290712525133064; visual box size=0.3576547495187927 0.31346256494802144 0.290712525133064
- link 9: geometry collision box size=0.2549993545935027 0.23179017415665532 0.37014261686751904; visual box size=0.2549993545935027 0.23179017415665532 0.37014261686751904
Joints:
- removed joint 0_10
- removed joint 0_13
- removed joint 0_4
- removed joint 0_7
- removed joint 10_11
- removed joint 11_12
- removed joint 13_14
- removed joint 14_15
- removed joint 2_3
- removed joint 5_6
- removed joint 7_8
- added joint 0_3: type revolute, parent 0, child 3, origin xyz=-0.3234541257224385 0 2 rpy=0 0 0, axis 0 0 1, limit lower=-3.14159 upper=3.14159 effort=0.0 velocity=0.0
- added joint 0_6: type revolute, parent 0, child 6, origin xyz=0 0.3032922543533117 2 rpy=0 0 0, axis 1 0 0, limit lower=-3.14159 upper=3.14159 effort=0.0 velocity=0.0
- added joint 0_8: type revolute, parent 0, child 8, origin xyz=0 -0.3032922543533117 2 rpy=0 0 0, axis 0 0 1, limit lower=-3.14159 upper=3.14159 effort=0.0 velocity=0.0
- added joint 3_4: type revolute, parent 3, child 4, origin xyz=-0.4027057677449959 0 0 rpy=0 0 0, axis 1 0 0, limit lower=-3.14159 upper=3.14159 effort=0.0 velocity=0.0
- added joint 6_7: type revolute, parent 6, child 7, origin xyz=0 0.41319882834782423 0 rpy=0 0 0, axis 1 0 0, limit lower=-3.14159 upper=3.14159 effort=0.0 velocity=0.0
- joint 0_1: axis 0 1 0 -> 0 0 1; origin xyz=0.2925562343733321 0 2 rpy=0 0 0 -> xyz=0.3234541257224385 0 2 rpy=0 0 0
- joint 1_2: axis 0 1 0 -> 1 0 0; origin xyz=0.3628604417647888 0 0 rpy=0 0 0 -> xyz=0.37282429908884995 0 0 rpy=0 0 0
- joint 4_5: axis 0 0 1 -> 1 0 0; origin xyz=0 0.24301260928841395 0 rpy=0 0 0 -> xyz=-0.19985707235031516 0 0.18808197727333587 rpy=0 0 0
- joint 8_9: origin xyz=0 -0.42683715933719335 0 rpy=0 0 0 -> xyz=0 -0.31346256494802144 0 rpy=0 0 0

Commit message: "Updated Asn 7"

File: body.urdf (robot description, URDF)
Before this commit: robot robot, 10 links, 9 joints
Links:
- removed link 7
- removed link 8
- removed link 9
- link 0: geometry collision box size=0.6226971482523986 0.8393749862805282 0.7866690631371045; visual box size=0.6226971482523986 0.8393749862805282 0.7866690631371045
- link 1: geometry collision box size=0.5373654882338088 0.9714915273767168 0.7101137113835942; visual box size=0.5373654882338088 0.9714915273767168 0.7101137113835942
- link 2: geometry collision box size=0.4376154040550936 0.4519822516459756 0.5457612360425445; visual box size=0.4376154040550936 0.4519822516459756 0.5457612360425445
- link 3: geometry collision box size=0.5317021123802037 0.5398169719545853 0.6870152877414296; visual box size=0.5317021123802037 0.5398169719545853 0.6870152877414296
- link 4: geometry collision box size=0.39913194534764 0.5373076935765515 0.36052808151476773; visual box size=0.39913194534764 0.5373076935765515 0.36052808151476773
- link 5: geometry collision box size=0.5947978005172063 0.569072517714698 0.5936296997144794; visual box size=0.5947978005172063 0.569072517714698 0.5936296997144794
- link 6: geometry collision box size=0.3257562601637994 0.33126266827862044 0.43409531435564913; visual box size=0.3257562601637994 0.33126266827862044 0.43409531435564913
Joints:
- removed joint 0_3
- removed joint 0_6
- removed joint 0_8
- removed joint 3_4
- removed joint 4_5
- removed joint 6_7
- removed joint 8_9
- added joint 1_3: type revolute, parent 1, child 3, origin xyz=-0.2686827441169044 0 0.3550568556917971 rpy=0 0 0, axis 0 0 1, limit lower=-3.14159 upper=3.14159 effort=0.0 velocity=0.0
- added joint 2_4: type revolute, parent 2, child 4, origin xyz=0 0.2259911258229878 -0.2728806180212722 rpy=0 0 0, axis 0 1 0, limit lower=-3.14159 upper=3.14159 effort=0.0 velocity=0.0
- added joint 2_5: type revolute, parent 2, child 5, origin xyz=0 0 -0.5457612360425445 rpy=0 0 0, axis 0 0 1, limit lower=-3.14159 upper=3.14159 effort=0.0 velocity=0.0
- added joint 3_6: type revolute, parent 3, child 6, origin xyz=0 0.26990848597729267 0.3435076438707148 rpy=0 0 0, axis 0 1 0, limit lower=-3.14159 upper=3.14159 effort=0.0 velocity=0.0
- joint 0_1: axis 0 0 1 -> 0 1 0; origin xyz=0.3234541257224385 0 2 rpy=0 0 0 -> xyz=-0.3113485741261993 0 2 rpy=0 0 0
- joint 1_2: origin xyz=0.37282429908884995 0 0 rpy=0 0 0 -> xyz=-0.2686827441169044 0 -0.3550568556917971 rpy=0 0 0
